File: ElleHacks-Soldering-Workshop/ElleHacks-Soldering-Workshop.kicad_sch (KiCad schematic)
At the start: 12 parts, among them J1 Power Input, Q1 2N3904, Q2 2N3904, U1 OS102011MA1QS1

Commit message: Dark Star
Parts:
- C1, C2: footprint (none) -> Library:WCAP-ATG8_5X11_DXL_
- D1, D2: footprint (none) -> Library:LEDRD254W57D500H1070
- J1: footprint (none) -> Library:691137710002
- R1, R2, R3, R4: footprint (none) -> Library:YAG_MF25_YAG
Changed lines of the file:
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@@
 			)
 		)
-		(property "Footprint" ""
+		(property "Footprint" "Library:LEDRD254W57D500H1070"
 			(at 130.81 44.45 0)
 			(effects
@@
 			)
 		)
-		(property "Footprint" ""
+		(property "Footprint" "Library:YAG_MF25_YAG"
 			(at 185.166 53.594 90)
 			(effects
@@
 			)
 		)
-		(property "Footprint" ""
+		(property "Footprint" "Library:WCAP-ATG8_5X11_DXL_"
 			(at 146.05 58.42 0)
 			(effects
@@
 			)
 		)
-		(property "Footprint" ""
+		(property "Footprint" "Library:LEDRD254W57D500H1070"
 			(at 184.15 44.45 0)
 			(effects
@@
 			)
 		)
-		(property "Footprint" ""
+		(property "Footprint" "Library:WCAP-ATG8_5X11_DXL_"
 			(at 172.72 58.42 0)
 			(effects
@@
 			)
 		)
-		(property "Footprint" ""
+		(property "Footprint" "Library:YAG_MF25_YAG"
 			(at 131.826 53.594 90)
 			(effects
@@
 			)
 		)
-		(property "Footprint" ""
+		(property "Footprint" "Library:YAG_MF25_YAG"
 			(at 152.146 48.514 90)
 			(effects
@@
 			)
 		)
-		(property "Footprint" ""
+		(property "Footprint" "Library:YAG_MF25_YAG"
 			(at 163.576 48.514 90)
 			(effects
@@
 			)
 		)
-		(property "Footprint" ""
+		(property "Footprint" "Library:691137710002"
 			(at 64.77 41.91 0)
 			(effects
